File: STM32G031J6M6/stm32G031J6M6-Breakout.brd (EAGLE design)
At the start: 29.1 x 36.5 mm, 10 parts, among them IC1 LDL112D33R, J2 PWR

Commit message: base code
Changed lines of the file:
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@@
 <wire x1="0" y1="36.54" x2="0" y2="0" width="0" layer="20"/>
 <text x="14.097" y="17.399" size="0.8128" layer="25" rot="R90">STM32G031</text>
-<text x="5.08" y="31.75" size="1.27" layer="1" rot="R90">VIN</text>
-<text x="7.62" y="31.75" size="1.27" layer="1" rot="R90">GND</text>
-<text x="10.16" y="31.75" size="1.27" layer="1" rot="R90">VDD</text>
-<text x="12.7" y="31.75" size="1.27" layer="1" rot="R90">JTCK</text>
-<text x="15.24" y="31.75" size="1.27" layer="1" rot="R90">JTMS</text>
-<text x="17.78" y="31.75" size="1.27" layer="1" rot="R90">P12</text>
-<text x="20.32" y="31.75" size="1.27" layer="1" rot="R90">PA8</text>
-<text x="22.86" y="31.75" size="1.27" layer="1" rot="R90">PA7</text>
-<text x="25.4" y="31.75" size="1.27" layer="1" rot="R90">NRST</text>
+<text x="5.08" y="31.75" size="1.27" layer="25" rot="R90">VIN</text>
+<text x="7.62" y="31.75" size="1.27" layer="25" rot="R90">GND</text>
+<text x="10.16" y="31.75" size="1.27" layer="25" rot="R90">VDD</text>
+<text x="12.7" y="31.75" size="1.27" layer="25" rot="R90">JTCK</text>
+<text x="15.24" y="31.75" size="1.27" layer="25" rot="R90">JTMS</text>
+<text x="17.78" y="31.75" size="1.27" layer="25" rot="R90">P12</text>
+<text x="20.32" y="31.75" size="1.27" layer="25" rot="R90">PA8</text>
+<text x="22.86" y="31.75" size="1.27" layer="25" rot="R90">PA7</text>
+<text x="25.4" y="31.75" size="1.27" layer="25" rot="R90">NRST</text>
 </plain>
 <attributes>
