File: Single-APA102c-Breakout/single-apa102c.brd (EAGLE design)
At the start: 13.9 x 10.5 mm, 5 parts

Commit message: base code
Parts:
- U$2: value CMD_C0DE_LOGOCMD_CODE_LOGO_TOP_COPPER -> CMD_C0DE_LOGOCMD_CODE_LOGO_SILK; device logos:CMD_C0DE_LOGO_TOP_COPPER -> logos:CMD_C0DE_LOGO_SILK
Changed lines of the file:
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@@
 <attribute name="NAME" x="9.37680625" y="8.368809375" size="0.4064" layer="25" font="vector" rot="R135" align="bottom-center"/>
 </element>
-<element name="U$2" library="logos" package="CMD_C0DE_LOGO_TOP_COPPER" value="CMD_C0DE_LOGOCMD_CODE_LOGO_TOP_COPPER" x="7.112" y="5.715" smashed="yes" rot="MR0"/>
+<element name="U$2" library="logos" package="CMD_C0DE_LOGO_SILK" value="CMD_C0DE_LOGOCMD_CODE_LOGO_SILK" x="7.112" y="5.715" smashed="yes" rot="MR0"/>
 <element name="J2" library="connector" package="1X04" value="" x="12.5" y="9.017" smashed="yes" rot="R270">
 <attribute name="NAME" x="14.3288" y="10.3632" size="1.27" layer="25" ratio="10" rot="R270"/>
